File: OBS-buttons-processor.sch (EAGLE design)
At the start: 23 parts

Commit message: initial prototype
Parts:
- removed BOARD1, BOARD2: (no value), SPCoast:BOARD100X50-NOHOLES
- removed CON1: (no value), SPCoast:CONNECTOR-M02508-LOCK
- removed J1, J2: (no value), SPCoast:CONNECTOR-M08LOCK
- removed LED1, LED2, LED3, LED4, LED5, LED6: (no value), SPCoast:LEDLED5MM
- removed SW1, SW2, SW3: (no value), SPCoast:SWITCH-SPSTPTH-508
- added R7: 10k, SPCoast:RPTH04
- R1, R2, R3, R4, R5, R6: value (none) -> 10k
Connections:
- removed net CUT: J1.3, SW1.O
- removed net CUT-LED: J2.1, R1.1
- removed net FADE: J1.4, SW1.S
- removed net FADE-LED: J2.6, R2.1
- removed net N$1: LED1.C, R1.2
- removed net N$2: LED2.C, R2.2
- removed net N$3: LED3.C, R3.2
- removed net N$4: LED4.C, R4.2
- removed net N$5: LED5.C, R5.2
- removed net N$6: LED6.C, R6.2
- removed net SCENE1: J1.5, SW2.O
- removed net SCENE1-LED: J2.2, R3.1
- removed net SCENE2: J1.6, SW2.S
- removed net SCENE2-LED: J2.5, R4.1
- removed net SCENE3: J1.7, SW3.O
- removed net SCENE3-LED: J2.3, R5.1
- removed net SCENE4: J1.8, SW3.S
- removed net SCENE4-LED: J2.4, R6.1
- removed net TRANSITION: CON1.B, J1.2
- net GND: no longer CON1.A, J2.7, J2.8, SW1.P, SW2.P, SW3.P
- net I1: now also R4.1
- net I2: now also R5.1
- net I3: now also R6.1
- net I4: now also R7.1
- net I5: now also R2.1
- net I6: now also R3.1
- net I7: now also R1.1
- net VCC: now also R1.2, R2.2, R3.2, R4.2, R5.2, R6.2, R7.2; no longer J1.1, LED1.A, LED2.A, LED3.A, LED4.A, LED5.A, LED6.A
Other:
- moved on the sheet: R1, R2, R3, R4, R5, R6
